File: output/pcbs/hasbii_pcb.kicad_pcb (KiCad board)
At the start: 2 copper layers, 160.9 x 104.5 mm, 56 parts

Commit message: output
Parts:
- moved MCU1 2.33 mm to (265.5, 116.0)
Connections:
- net CL renamed P7
- net CS renamed P14
- net DA renamed P6
- D19 pad 1: r2 -> t2
- D19 pad 2: c5_r2 -> c5_t2
- D20 pad 1: r2 -> t2
- D20 pad 2: c4_r2 -> c4_t2
- D21 pad 1: r2 -> t2
- D21 pad 2: c3_r2 -> c3_t2
- D22 pad 1: r2 -> t2
- D22 pad 2: c2_r2 -> c2_t2
- D23 pad 1: r1 -> t1
- D23 pad 2: c2_r1 -> c2_t1
- D24 pad 1: r2 -> t2
- D24 pad 2: c1_r2 -> c1_t2
- D25 pad 1: r1 -> t1
- D25 pad 2: c1_r1 -> c1_t1
- MCU1 pad 13: r0 -> t2
- MCU1 pad 18: P19 -> t1
- S19 pad 1: c5_r2 -> c5_t2
- S20 pad 1: c4_r2 -> c4_t2
- S21 pad 1: c3_r2 -> c3_t2
- S22 pad 1: c2_r2 -> c2_t2
- S23 pad 1: c2_r1 -> c2_t1
- S24 pad 1: c1_r2 -> c1_t2
- S25 pad 1: c1_r1 -> c1_t1
Routing:
- net c2_t2: track 0.00 -> 8.27 mm, vias 0 -> 1
- net c2_r2: track 16.5 -> 8.27 mm, vias 2 -> 1
- net c2_r1: track 16.5 -> 8.27 mm, vias 2 -> 1
- net c2_t1: track 0.00 -> 8.27 mm, vias 0 -> 1
- net c5_t2: track 0.00 -> 8.27 mm, vias 0 -> 1
- net c5_r2: track 16.5 -> 8.27 mm, vias 2 -> 1
- net c4_t2: track 0.00 -> 8.27 mm, vias 0 -> 1
- net c4_r2: track 16.5 -> 8.27 mm, vias 2 -> 1
- net c3_r2: track 16.5 -> 8.27 mm, vias 2 -> 1
- net c3_t2: track 0.00 -> 8.27 mm, vias 0 -> 1
- net c1_t2: track 0.00 -> 8.27 mm, vias 0 -> 1
- net c1_t1: track 0.00 -> 8.27 mm, vias 0 -> 1
- net c1_r1: track 16.5 -> 8.27 mm, vias 2 -> 1
- net c1_r2: track 16.5 -> 8.27 mm, vias 2 -> 1
