File: output/pcbs/hasbii_pcb.kicad_pcb (KiCad board)
At the start: 2 copper layers, 160.9 x 104.5 mm, 56 parts

Commit message: feat: remove reset switch and reposition TRRS jack
Remove reset_switch footprint from config (will be added manually in KiCad).
Adjust TRRS jack anchor shift and rotation for better board placement.

Co-Authored-By: Claude Sonnet 4.6 <noreply@anthropic.com>
Parts:
- added DISP1: , ceoloide:display_ssd1306, F.Cu at (265.5, 119.5)
- added TRRS1: , ceoloide:trrs_pj320a (reversible, symmetric), F.Cu at (274.4, 146.0)
Connections:
- MCU1 pad 10: P7 -> c6
- MCU1 pad 102: P0 -> DATA
- MCU1 pad 11: c5 -> SDA
- MCU1 pad 12: c6 -> SCL
- MCU1 pad 13: t2 -> P10
- MCU1 pad 14: c4 -> P16
- MCU1 pad 16: c2 -> t1
- MCU1 pad 17: c3 -> t2
- MCU1 pad 18: t1 -> r3
- MCU1 pad 19: P20 -> r2
- MCU1 pad 20: P21 -> r1
- MCU1 pad 6: r1 -> c2
- MCU1 pad 7: r2 -> c3
- MCU1 pad 8: r3 -> c4
- MCU1 pad 9: P6 -> c5
Routing:
- net DISP1_4: track 0.00 -> 3.50 mm
- net DISP1_3: track 0.00 -> 3.50 mm
- net DISP1_2: track 0.00 -> 3.50 mm
- net DISP1_1: track 0.00 -> 3.50 mm

Commit message: feat: add case outlines and STL generation to config
Add switch cutouts, mounting plate, and top frame outlines. Add cases
section to generate mounting_plate (1.5mm), bottom_plate (1.6mm), and
top_frame (3mm) STL files via Ergogen.

Co-Authored-By: Claude Sonnet 4.6 <noreply@anthropic.com>
Parts:
- moved TRRS1 4.00 mm to (274.4, 142.0)
Changed lines of the file:
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@@
   (footprint "ceoloide:trrs_pj320a (reversible, symmetric)"
     (layer "F.Cu")
-    (at 274.39 146 -90)
+    (at 274.39 142 -90)
     (property "Reference" "TRRS1"
       (at 0 14.2 -90)
